File: KiCAD/main/_autosave-main.kicad_pcb (KiCad board)
At the start: 2 copper layers, 57.5 x 267.7 mm, 153 parts, among them J1 USB_C_Receptacle_USB2.0_14P, J2 Conn_Coaxial, SW1 SW_SPDT, SW2 SW_Push, SW3 SW_Push, U1 SX1262IMLTRT, U2 TP4056-42-ESOP8, U3 TLV75533PDRV, U4 ESP32-S3-MINI-1, U5 BGS12WN6E6327, U6 FT231XQ, U7 CH340X

Commit message: rev 2!
Parts:
- removed the BT1 at (351.6, 107.9)
- removed the BT1 at (331.2, -53.8)
- removed the BT1 at (358.9, 18.5)
- removed BZ1: Buzzer, Buzzer_Beeper:Buzzer_CUI_CPT-9019S-SMT
- removed the C1 at (374.0, -63.6)
- removed the C1 at (354.9, 115.4)
- removed the C1 at (367.6, 15.7)
- removed the C10 at (358.0, -106.4)
- removed the C10 at (364.9, -10.5)
- removed the C10 at (346.7, 100.5)
- removed the C11 at (360.5, -11.8)
- removed the C11 at (356.8, -109.7)
- removed the C11 at (346.6, 97.6)
- removed the C12 at (360.5, -17.4)
- removed the C12 at (353.1, 97.4)
- removed the C12 at (364.2, -112.2)
- removed the C13 at (357.1, 98.4)
- removed the C13 at (361.5, -21.3)
- removed the C13 at (369.5, -111.2)
- removed the C15 at (363.1, 9.15)
- removed the C15 at (344.8, -51.9)
- removed the C15 at (356.7, 107.1)
- removed the C16 at (361.6, 14.3)
- removed the C16 at (347.8, -51.9)
- removed the C16 at (356.3, 115.5)
- removed the C17 at (368.9, 20.0)
- removed the C17 at (358.7, 123.6)
- removed the C17 at (364.0, -62.9)
- removed the C18 at (356.7, 123.6)
- removed the C18 at (366.8, -64.4)
- removed the C18 at (371.1, 21.1)
- removed C19 (x2), C9 (x2): 0.1uF, Capacitor_SMD:C_01005_0402Metric
- removed the C2 at (365.1, 13.5)
- removed the C2 at (353.6, 112.9)
- removed the C2 at (373.5, -64.9)
- removed C20 (x2), C21 (x2): 47uF, Capacitor_SMD:C_01005_0402Metric
- removed the C3 at (370.0, -86.4)
- removed the C3 at (374.0, 104.5)
- removed the C3 at (373.0, -8.75)
- removed the C4 at (373.1, -9.90)
- removed the C4 at (372.5, -86.9)
- removed the C4 at (373.9, 103.2)
- removed the C5 at (357.7, -107.5)
- removed the C5 at (362.7, -10.7)
- removed the C6 at (362.8, -111.5)
- removed the C6 at (360.0, -15.4)
- removed the C6 at (351.0, 96.8)
- removed the C7 at (346.7, 99.7)
- removed the C7 at (363.5, -10.8)
- removed the C7 at (357.8, -108.2)
- removed C8 (x2): 10uF, Capacitor_SMD:C_01005_0402Metric
- removed the D1 at (364.2, -58.9)
- removed the D1 at (361.9, 15.5)
- removed the D1 at (351.4, 118.4)
- removed the D2 at (355.0, 108.2)
- removed the D2 at (361.4, 16.7)
- removed the D2 at (370.0, -59.6)
- removed D3 (x3), D4 (x3), D5 (x3): LED, LED_SMD:LED_0402_1005Metric
- removed the FL1 at (354.7, 100.1)
- removed the FL1 at (367.2, -109.8)
- removed the FL1 at (363.1, -19.5)
- removed the G*** at (398.6, 43.6)
- removed the G*** at (374.7, 93.3)
- removed the G*** at (368.5, -15.6)
- removed the G*** at (189.6, -169.1)
- removed the J1 at (361.1, -52.9)
- removed the J1 at (366.0, 30.5)
- removed the J1 at (349.8, 129.3)
- removed the J2 at (371.4, -121.7)
- removed the J2 at (363.8, -27.9)
- removed the J2 at (361.7, 94.0)
- removed the L1 at (361.6, -10.8)
- removed the L1 at (347.4, 97.5)
- removed the L1 at (358.0, -109.0)
- removed the L2 at (365.2, -111.7)
- removed the L2 at (361.0, -19.2)
- removed the L2 at (353.5, 98.1)
- removed the R1 at (355.3, 128.0)
- removed the R1 at (360.2, 29.3)
- removed the R1 at (354.8, -54.2)
- removed the R10 at (360.0, -59.2)
- removed the R10 at (365.3, 24.2)
- removed R11: 270R, Resistor_SMD:R_01005_0402Metric
- removed R12 (x3): 1K, Resistor_SMD:R_01005_0402Metric
- removed the R2 at (355.1, 131.4)
- removed the R2 at (367.5, -54.2)
- removed the R2 at (371.8, 29.3)
- removed R3 (x3), R8 (x3): 10K, Resistor_SMD:R_01005_0402Metric
- removed the R4 at (359.5, -105.2)
- removed the R4 at (347.6, 102.7)
- removed the R4 at (366.3, -13.2)
- removed the R5 at (370.5, -112.2)
- removed the R5 at (360.3, -21.6)
- removed the R5 at (357.2, 99.6)
- removed R6 (x3): 2K, Resistor_SMD:R_01005_0402Metric
- removed the R7 at (342.8, -55.7)
- removed the R7 at (358.1, 107.1)
- removed the R7 at (354.4, 11.5)
- removed the R9 at (361.8, -59.2)
- removed the R9 at (366.3, 24.2)
- removed the SW1 at (346.6, 117.3)
- removed the SW1 at (373.2, -58.6)
- removed the SW1 at (354.6, 3.20)
- removed SW2 (x3): SW_Push, Button_Switch_SMD:SW_SPST_PTS810
- removed SW3 (x3): SW_Push, Button_Switch_SMD:SW_SPST_PTS645Sx43SMTR92
- removed the U1 at (363.0, -14.4)
- removed the U1 at (361.8, -108.4)
- removed the U1 at (350.1, 100.0)
- removed the U2 at (358.6, 11.5)
- removed the U2 at (347.0, -55.7)
- removed the U2 at (358.2, 111.3)
- removed the U3 at (365.9, 15.3)
- removed the U3 at (353.2, 114.8)
- removed the U3 at (371.4, -65.8)
- removed the U4 at (370.9, -0.45)
- removed the U4 at (369.7, -78.0)
- removed the U4 at (371.9, 113.1)
- removed U5 (x3): BGS12WN6E6327, Package_LGA:Infineon_PG-TSNP-6-10_0.7x1.1mm_0.7x1.1mm_P0.4mm
- removed the U6 at (360.7, -63.2)
- removed the U6 at (365.5, 20.3)
- added BT1: Battery_Cell, Connector_JST:JST_PH_S2B-PH-K_1x02_P2.00mm_Horizontal, F.Cu at (96.6, 69.7)
- added C1: 1uF, Capacitor_SMD:C_0603_1608Metric, F.Cu at (94.8, 81.8)
- added C10: 0.1uF, Capacitor_SMD:C_0402_1005Metric, F.Cu at (94.6, 47.5)
- added C11: 0.1uF, Capacitor_SMD:C_0402_1005Metric, F.Cu at (95.6, 42.9)
- added C12: 22 pF, Capacitor_SMD:C_0603_1608Metric, F.Cu at (100.7, 42.1)
- added C13: 100nF, Capacitor_SMD:C_0402_1005Metric, F.Cu at (104.9, 41.5)
- added C15: 10uF, Capacitor_SMD:C_0603_1608Metric, F.Cu at (101.0, 84.9)
- added C16: 10uF, Capacitor_SMD:C_0603_1608Metric, F.Cu at (91.8, 75.8)
- added C17: 0.1uF, Capacitor_SMD:C_0402_1005Metric, F.Cu at (106.2, 76.2)
- added C18: 0.1uF, Capacitor_SMD:C_0402_1005Metric, F.Cu at (101.2, 76.0)
- added C2: 1uF, Capacitor_SMD:C_0603_1608Metric, F.Cu at (99.8, 80.1)
- added C3: 0.1uf, Capacitor_SMD:C_0402_1005Metric, F.Cu at (104.9, 50.2)
- added C4: 22uF, Capacitor_SMD:C_0805_2012Metric, F.Cu at (103.4, 48.6)
- added C5: 470pF, Capacitor_SMD:C_0603_1608Metric, F.Cu at (101.4, 78.9)
- added C6: 0.1uF, Capacitor_SMD:C_0402_1005Metric, F.Cu at (97.2, 42.4)
- added C7: 0.1uF, Capacitor_SMD:C_0402_1005Metric, F.Cu at (94.6, 45.0)
- added D1: D_Schottky, Diode_SMD:D_SOD-323, F.Cu at (97.5, 84.0)
- added D2: D_Schottky, Diode_SMD:D_SOD-323, F.Cu at (94.3, 76.2)
- added FL1: 0900FM15K0039, RF_Converter:Balun_Johanson_0900FM15K0039, F.Cu at (104.8, 45.8)
- added J1: USB_C_Receptacle_USB2.0_14P, Connector_USB:USB_C_Receptacle_GCT_USB4110, F.Cu at (102.2, 90.5)
- added J2: Conn_Coaxial, Connector_Coaxial:SMA_Amphenol_132289_EdgeMount, F.Cu at (100.3, 32.9)
- added L1: 15uH, Inductor_SMD:L_0805_2012Metric, F.Cu at (95.7, 41.0)
- added L2: 18 nH, Inductor_SMD:L_0603_1608Metric, F.Cu at (103.2, 42.7)
- added R1: 5K1, Resistor_SMD:R_0603_1608Metric, F.Cu at (100.2, 83.3)
- added R10: 10K, Resistor_SMD:R_0603_1608Metric, F.Cu at (93.1, 48.9)
- added R2: 5K1, Resistor_SMD:R_0603_1608Metric, F.Cu at (105.3, 83.3)
- added R4: 10K, Resistor_SMD:R_0603_1608Metric, F.Cu at (97.1, 49.6)
- added R5: 100R, Resistor_SMD:R_0402_1005Metric, F.Cu at (102.7, 40.1)
- added R7: 1.2K, Resistor_SMD:R_0603_1608Metric, F.Cu at (100.8, 74.6)
- added R9: 10K, Resistor_SMD:R_0603_1608Metric, F.Cu at (93.1, 45.4)
- added SW1: SW_SPDT, customlib:SSSS810701, F.Cu at (91.7, 82.5)
- added U1: SX1262IMLTRT, Package_DFN_QFN:QFN-24-1EP_4x4mm_P0.5mm_EP2.6x2.6mm, F.Cu at (98.8, 46.0)
- added U2: TP4056-42-ESOP8, Package_SO:SOIC-8-1EP_3.9x4.9mm_P1.27mm_EP2.41x3.3mm_ThermalVias, F.Cu at (102.7, 70.8)
- added U3: BGS12P2L, Package_LGA:Infineon_PG-TSNP-6-10_0.7x1.1mm_0.7x1.1mm_P0.4mm, F.Cu at (107.0, 43.6)
- added U4: ESP32-S3-MINI-1, RF_Module:ESP32-S2-MINI-1, F.Cu at (102.8, 58.7)
- added U6: MIC5219-3.3YMM, Package_SO:MSOP-8_3x3mm_P0.65mm, F.Cu at (97.2, 77.7)
- C14: footprint Capacitor_SMD:C_01005_0402Metric -> Capacitor_SMD:C_0603_1608Metric
- moved U7 258.6 mm to (104.0, 79.1)
- moved C14 258.3 mm to (99.2, 40.1), turned to -135 degrees
Routing:
- net V-: track 823.3 -> 259.0 mm, vias 26 -> 15
- net VCC: track 348.8 -> 108.9 mm, vias 25 -> 4
- net Net-(U4-EN): track 108.6 -> 0.00 mm, vias 6 -> 0
- net Net-(U4-IO10): track 83.1 -> 0.00 mm, vias 4 -> 0
- net V+: track 121.6 -> 50.0 mm, vias 5 -> 4
- net CHRG: track 69.8 -> 0.00 mm, vias 3 -> 0
- net Net-(SW1-A): track 47.2 -> 5.09 mm
- net SERIAL_N: track 51.8 -> 13.5 mm, vias 0 -> 2
- net SPI_CS: track 42.1 -> 4.62 mm
- net SPI_CLK: track 40.7 -> 3.87 mm
- net SERIAL_P: track 49.3 -> 13.5 mm, vias 0 -> 2
- net Net-(D1-K): track 49.7 -> 14.5 mm
- net ~{STDBY}: track 0.00 -> 34.4 mm, vias 0 -> 2
- net CHRG_BAT: track 0.00 -> 31.6 mm
- net ~{CHRG}: track 0.00 -> 28.7 mm, vias 0 -> 2
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- added copper zone on F.Cu, net V-
- removed copper zone on B.Cu, net V-
Other:
- board size 57.5 x 267.7 mm -> 19.6 x 63.9 mm
- board text removed: "VIP(E)R Rev1.0"
- board text removed: "VIP(E)R Rev1.1"
