File: KiCAD/main/finals/rev1.1/main.kicad_pcb (KiCad board)
At the start: 2 copper layers, 29.8 x 66.1 mm, 52 parts, among them J1 USB_C_Receptacle_USB2.0_14P, J2 Conn_Coaxial, SW1 SW_SPDT, SW2 SW_Push, SW3 SW_Push, U1 SX1262IMLTRT, U2 TP4056-42-ESOP8, U3 TLV75533PDRV, U4 ESP32-S3-MINI-1, U5 BGS12WN6E6327, U6 FT231XQ

Commit message: rev 2!
Parts:
- added G***: LOGO, customlib:viper, F.Cu at (16.0, 15.3)
- moved G*** 21.9 mm to (151.1, 63.7)
- moved C19 20.8 mm to (149.6, 101.2)
- moved SW3 20.8 mm to (154.4, 92.4)
- moved C12 20.8 mm to (142.4, 60.8)
- moved J2 20.8 mm to (145.6, 50.3)
- moved SW2 20.8 mm to (139.1, 73.2)
- moved U1 20.8 mm to (144.9, 63.9)
- moved U5 20.8 mm to (145.6, 56.4)
- moved C10 20.8 mm to (146.7, 67.7)
- moved C20 20.8 mm to (149.0, 102.8)
- moved C21 20.8 mm to (146.4, 102.8)
- moved C4 20.8 mm to (154.9, 68.3)
- moved L2 20.8 mm to (142.9, 59.0)
- moved R3 20.8 mm to (154.8, 86.5)
- moved R7 20.8 mm to (136.3, 89.7)
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Routing:
- net DIO2: track 0.00 -> 24.7 mm, vias 0 -> 2
- net VCC: track 90.0 -> 88.2 mm
- added copper zone on F.Cu, net V-
Other:
- board size 29.8 x 66.1 mm -> 23.7 x 66.1 mm
